Commit message: master

File: carmodel_description/urdf/carmodel2.urdf (robot description, URDF)
Before this commit: robot carmodel, 6 links, 5 joints
Links:
- removed link odom
- added link base_footprint; collision box size=0.001 0.001 0.001; visual box size=0.001 0.001 0.001
- added link base_scan
- link base_link: geometry collision box size=0.5 0.3 0.07; visual mesh filename=package://carmodel_description/meshes/Body_with_radar.STL
Joints:
- removed joint base_odom
- added joint base_footprint_joint: type fixed, parent base_footprint, child base_link, origin xyz=0 0 0.017 rpy=0 0 0
- added joint scan_joint: type fixed, parent base_link, child base_scan, origin xyz=0 0 0.122 rpy=0 0 0
- joint joint_base_wheel1: limit effort=500 velocity=500 -> (none)
- joint joint_base_wheel2: limit effort=500 velocity=500 -> (none)
- joint joint_base_wheel3: limit effort=500 velocity=500 -> (none)
- joint joint_base_wheel4: limit effort=500 velocity=500 -> (none)

File: carmodel_description/urdf/carmodel2.urdf.xacro (robot description, xacro)
@@ -1,9 +1,9 @@
 <?xml version="1.0"?>
 <robot name="carmodel" xmlns:xacro="http://ros.org/wiki/xacro">
-<xacro:include filename="$(find carmodel_description)/urdf/carmodel2.urdf"/>
-<xacro:property name="wheel_radius" value="0.03018"/>
-<xacro:property name="width" value="0.13189"/>
+  <xacro:include filename="$(find carmodel_description)/urdf/carmodel2.urdf"/>
+  <xacro:property name="wheel_radius" value="0.03018"/>
+  <xacro:property name="width" value="0.13189"/>
     <gazebo reference="base_link">
-      <material>Gazebo/Black</material>
+      <material>Gazebo/Orange</material>
     </gazebo>
     <gazebo reference="wheel_1">
@@ -59,3 +59,59 @@
     </plugin>
   </gazebo>
+  <gazebo>
+    <plugin name="differential_drive_controller" filename="libgazebo_ros_diff_drive.so">
+      <rosDebugLevel>na</rosDebugLevel>
+      <publishWheelTF>true</publishWheelTF>
+      <robotNamespace>/</robotNamespace>
+      <publishTf>true</publishTf>
+      <publishWheelJointState>true</publishWheelJointState>
+      <alwaysOn>true</alwaysOn>
+      <updateRate>30.0</updateRate>
+      <legacyMode>true</legacyMode>
+      <leftJoint>joint_base_wheel1</leftJoint>
+      <rightJoint>joint_base_wheel3</rightJoint>
+      <wheelSeparation>${width*2}</wheelSeparation>
+      <wheelDiameter>${2*wheel_radius}</wheelDiameter>
+      <broadcastTF>1</broadcastTF>
+      <wheelTorque>50</wheelTorque>
+      <wheelAcceleration>1.8</wheelAcceleration>
+      <commandTopic>cmd_vel</commandTopic>
+      <odometryFrame>odom</odometryFrame>
+      <odometryTopic>odom</odometryTopic>
+      <odometrySource>world</odometrySource>
+      <robotBaseFrame>base_footprint</robotBaseFrame>
+    </plugin>
+  </gazebo>
+  <gazebo reference="base_scan">
+    <sensor type="ray" name="lds_lfcd_sensor">
+    <pose>0 0 0 0 0 0</pose>
+    <visualize>false</visualize>
+    <update_rate>5.0</update_rate>
+    <ray>
+      <scan>
+        <horizontal>
+        <samples>360</samples>
+        <resolution>1</resolution>
+        <min_angle>0.0</min_angle>
+        <max_angle>6.28319</max_angle>
+        </horizontal>
+      </scan>
+      <range>
+        <min>0.120</min>
+        <max>3.5</max>
+        <resolution>0.015</resolution>
+      </range>
+      <noise>
+        <type>gaussian</type>
+        <mean>0.0</mean>
+        <stddev>0.01</stddev>
+      </noise>
+    </ray>
+    <plugin name="gazebo_ros_lds_lfcd_controller" filename="libgazebo_ros_laser.so">
+      <topicName>/scan</topicName>
+      <frameName>base_scan</frameName>
+    </plugin>
+    </sensor>
+  </gazebo>
+  <carmodel/>
 </robot>

Commit message: Update robot model

File: carmodel_description/urdf/carmodel2.urdf (robot description, URDF)
Before this commit: robot carmodel, 7 links, 6 joints
Links:
- link base_link: mass 32 -> 65.8282; geometry collision box size=0.5 0.3 0.07; visual mesh filename=package://carmodel_description/meshes/Body3.STL
